File: hardware/pcb_source/universal_oled.kicad_pcb (KiCad board)
At the start: 2 copper layers, 30 x 36.5 mm, 14 parts, among them J1 Conn_01x06, J2 Conn_01x02, J3 Conn_01x04, J5 Conn_01x03, J6 Conn_01x06, U2 ESP32-C3-WROOM-02, U3 TLV70235_SOT23-5

Commit message: New PCB version
Parts:
- removed J1: Conn_01x06, Connector_PinHeader_2.54mm:PinHeader_1x06_P2.54mm_Vertical
- J2: value Conn_01x02 -> Conn_01x04; footprint Connector_JST:JST_XH_B2B-XH-A_1x02_P2.50mm_Vertical -> Connector_JST:JST_XH_B4B-XH-A_1x04_P2.50mm_Vertical
- moved J5 3.02 mm to (162.3, 73.9)
- moved J2 0.16 mm to (148.9, 73.4), turned to 0 degrees
Connections:
- J2 pad 2: +5V -> D+
- U2 pad 13: unconnected-(U2-IO18-Pad13) -> D-
- U2 pad 14: unconnected-(U2-IO19-Pad14) -> D+
Routing:
- net D+: track 0.00 -> 34.9 mm, vias 0 -> 1
- net TX: track 34.6 -> 0.00 mm, vias 1 -> 0
- net RX: track 33.7 -> 0.00 mm, vias 1 -> 0
- net D-: track 0.00 -> 32.7 mm, vias 0 -> 1
- net VCC: track 68.0 -> 58.7 mm
- net Net-(J6-Pin_5): track 25.7 -> 18.3 mm
- net Net-(J6-Pin_4): track 37.4 -> 32.9 mm, vias 2 -> 0
- net Net-(J6-Pin_6): track 27.9 -> 24.2 mm
- net Net-(J5-Pin_2): track 25.6 -> 28.3 mm, vias 0 -> 1
- net SDA: track 25.6 -> 23.0 mm
- net Net-(J6-Pin_1): track 31.6 -> 33.5 mm
- net Net-(J6-Pin_3): track 31.2 -> 29.5 mm
- net SCL: track 22.3 -> 23.7 mm
- net +5V: track 19.0 -> 20.1 mm
- net GND: vias 10 -> 44
Other:
- board text added: "GND D+ D- VCC"
- board text added: "VCC D- D+ GND"
- board text added: "VCC DIO GND"
- board text removed: "-"
- board text removed: "GND X VCC RX TX X"
- board text removed: "X TX RX VCC X GND"
